File: KiCAD/8DIN2VGA/8DIN2VGA.kicad_pcb (KiCad board)
At the start: 2 copper layers, 39.8 x 17.6 mm, 7 parts, among them P1 8_pin_DIN_Landing, P2 VGA, P3 3.5mm_vertical

Commit message: Update with new 5V design
Parts:
- moved G*** 0.37 mm to (145.6, 99.6)
Other:
- board size 39.8 x 17.6 mm -> 39.7 x 17.5 mm
Changed lines of the file:
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@@
-(kicad_pcb (version 20171130) (host pcbnew "(5.1.8-0-10_14)")
+(kicad_pcb (version 20171130) (host pcbnew "(5.1.10-1-10_14)")
   (general
     (thickness 1.6002)
@@
     (38 B.Mask user)
     (39 F.Mask user)
-    (42 Eco1.User user hide)
+    (42 Eco1.User user)
     (43 Eco2.User user hide)
     (44 Edge.Cuts user)
@@
     (user_trace_width 0.762)
     (trace_clearance 0.16)
-    (zone_clearance 0.19)
+    (zone_clearance 0.16)
     (zone_45_only no)
     (trace_min 0.1524)
@@
   )
   (module 8DIN2VGA:RD_logo (layer Front)
-    (at 145.4 99.87 270)
+    (at 145.63 99.58 270)
     (fp_text reference G*** (at -4.13 -7.58 90) (layer F.SilkS) hide
       (effects (font (size 1.524 1.524) (thickness 0.3)))
@@
       (effects (font (size 1 1) (thickness 0.25)))
     )
+    (fp_text user G*** (at -16.34 -15.37) (layer F.Fab) hide
+      (effects (font (size 1.524 1.524) (thickness 0.3)))
+    )
     (fp_poly (pts (xy 3.574517 -9.727315) (xy 3.264266 -9.727315) (xy 3.269914 -7.631346) (xy 3.275563 -5.535378)
       (xy 3.465884 -5.539956) (xy 3.560978 -5.540384) (xy 3.645487 -5.537475) (xy 3.704704 -5.53183)
@@
       (xy -3.563235 -18.851141) (xy -3.562818 -18.856478) (xy -3.551239 -18.93952) (xy 3.574517 -18.93952)
       (xy 3.574517 -9.727315)) (layer Eco2.User) (width 0.01))
-    (fp_text user G*** (at -16.34 -15.37) (layer F.Fab) hide
-      (effects (font (size 1.524 1.524) (thickness 0.3)))
-    )
-    (pad 4 smd roundrect (at -3.36 -3.73 270) (size 1.2 2) (layers Front F.Mask) (roundrect_rratio 0.125)
+    (pad 4 smd roundrect (at -3.36 -3.48 270) (size 1.2 2) (layers Front F.Mask) (roundrect_rratio 0.125)
       (net 11 GND) (zone_connect 2))
-    (pad 4 smd roundrect (at -3.36 -3.73 270) (size 1.2 2) (layers Back B.Mask) (roundrect_rratio 0.125)
+    (pad 4 smd roundrect (at -3.36 -3.48 270) (size 1.2 2) (layers Back B.Mask) (roundrect_rratio 0.125)
       (net 11 GND) (zone_connect 2))
     (pad 3 smd roundrect (at 3.33 -0.33 270) (size 1.2 2) (layers Back B.Mask) (roundrect_rratio 0.125)
@@
       (effects (font (size 1 1) (thickness 0.15)) (justify mirror))
     )
+    (fp_line (start -2.905 -5.06) (end 27.895 -5.06) (layer Dwgs.User) (width 0.12))
+    (fp_line (start -2.905 3.91) (end 27.895 3.91) (layer Dwgs.User) (width 0.12))
+    (fp_line (start -2.905 3.91) (end -2.905 -5.06) (layer Dwgs.User) (width 0.12))
+    (fp_line (start 27.895 3.91) (end 27.895 -5.06) (layer Dwgs.User) (width 0.12))
+    (fp_line (start 19.33 -5.08) (end 19.33 -9.33) (layer Dwgs.User) (width 0.12))
+    (fp_line (start 19.33 -9.33) (end 7.28 -9.33) (layer Dwgs.User) (width 0.12))
     (fp_line (start 7.28 -9.33) (end 7.28 -5.04) (layer Dwgs.User) (width 0.12))
-    (fp_line (start 19.33 -9.33) (end 7.28 -9.33) (layer Dwgs.User) (width 0.12))
-    (fp_line (start 19.33 -5.08) (end 19.33 -9.33) (layer Dwgs.User) (width 0.12))
-    (fp_line (start 27.895 3.91) (end 27.895 -5.06) (layer Dwgs.User) (width 0.12))
-    (fp_line (start -2.905 3.91) (end -2.905 -5.06) (layer Dwgs.User) (width 0.12))
-    (fp_line (start -2.905 3.91) (end 27.895 3.91) (layer Dwgs.User) (width 0.12))
-    (fp_line (start -2.905 -5.06) (end 27.895 -5.06) (layer Dwgs.User) (width 0.12))
     (pad 1 thru_hole rect (at 17.075 1.98) (size 1.7 1.7) (drill 1) (layers *.Cu *.Mask)
       (net 4 /RED) (zone_connect 2))
@@
       (net 11 GND) (zone_connect 1))
     (pad 2 thru_hole circle (at 14.785 1.98) (size 1.7 1.7) (drill 1) (layers *.Cu *.Mask)
-      (net 5 /GREEN) (zone_connect 2))
+      (net 5 /GREEN))
     (pad 3 thru_hole circle (at 12.495 1.98) (size 1.7 1.7) (drill 1) (layers *.Cu *.Mask)
-      (net 6 /BLUE) (zone_connect 2))
-    (pad 4 thru_hole circle (at 10.205 1.98) (size 1.7 1.7) (drill 1) (layers *.Cu *.Mask)
-      (zone_connect 2))
+      (net 6 /BLUE))
+    (pad 4 thru_hole circle (at 10.205 1.98) (size 1.7 1.7) (drill 1) (layers *.Cu *.Mask))
     (pad 5 thru_hole circle (at 7.915 1.98) (size 1.7 1.7) (drill 1) (layers *.Cu *.Mask)
-      (net 11 GND) (zone_connect 2))
+      (net 11 GND))
     (pad 6 thru_hole circle (at 18.22 0) (size 1.7 1.7) (drill 1) (layers *.Cu *.Mask)
-      (net 11 GND) (zone_connect 2))
+      (net 11 GND))
     (pad 7 thru_hole circle (at 15.93 0) (size 1.7 1.7) (drill 1) (layers *.Cu *.Mask)
-      (net 11 GND) (zone_connect 2))
+      (net 11 GND))
     (pad 8 thru_hole circle (at 13.64 0) (size 1.7 1.7) (drill 1) (layers *.Cu *.Mask)
-      (net 11 GND) (zone_connect 2))
+      (net 11 GND))
     (pad 9 thru_hole circle (at 11.35 0) (size 1.7 1.7) (drill 1) (layers *.Cu *.Mask)
-      (net 12 /+5V) (zone_connect 2))
+      (net 12 /+5V))
     (pad 10 thru_hole circle (at 9.06 0) (size 1.7 1.7) (drill 1) (layers *.Cu *.Mask)
-      (net 11 GND) (zone_connect 2))
-    (pad 11 thru_hole circle (at 17.075 -1.98) (size 1.7 1.7) (drill 1) (layers *.Cu *.Mask)
-      (zone_connect 2))
+      (net 11 GND))
+    (pad 11 thru_hole circle (at 17.075 -1.98) (size 1.7 1.7) (drill 1) (layers *.Cu *.Mask))
     (pad 12 thru_hole circle (at 14.785 -1.98) (size 1.7 1.7) (drill 1) (layers *.Cu *.Mask)
-      (net 1 /Audio_L_VGA) (zone_connect 2))
+      (net 1 /Audio_L_VGA))
     (pad 13 thru_hole circle (at 12.495 -1.98) (size 1.7 1.7) (drill 1) (layers *.Cu *.Mask)
-      (net 8 /SYNC) (zone_connect 2))
-    (pad 14 thru_hole circle (at 10.205 -1.98) (size 1.7 1.7) (drill 1) (layers *.Cu *.Mask)
-      (zone_connect 2))
+      (net 8 /SYNC))
+    (pad 14 thru_hole circle (at 10.205 -1.98) (size 1.7 1.7) (drill 1) (layers *.Cu *.Mask))
     (pad 15 thru_hole circle (at 7.915 -1.98) (size 1.7 1.7) (drill 1) (layers *.Cu *.Mask)
-      (net 2 "Net-(C2-Pad2)") (zone_connect 2))
+      (net 2 "Net-(C2-Pad2)"))
     (model "${KIPRJMOD}/Materials/VGA Female Slim.step"
       (offset (xyz -2.9 -5.05 0))
@@
     (effects (font (size 0.393701 0.393701) (thickness 0.098425)))
   )
-  (gr_line (start 158.88 112.44) (end 156.86 114.46) (layer Edge.Cuts) (width 0.1))
-  (gr_line (start 158.88 98) (end 158.88 112.44) (layer Edge.Cuts) (width 0.1))
-  (gr_line (start 151.18 98) (end 158.88 98) (layer Edge.Cuts) (width 0.1))
-  (gr_line (start 151.18 107.25) (end 151.18 98) (layer Edge.Cuts) (width 0.1))
-  (gr_line (start 150.1 107.25) (end 151.18 107.25) (layer Edge.Cuts) (width 0.1))
-  (gr_line (start 150.1 96.82) (end 150.1 107.25) (layer Edge.Cuts) (width 0.1))
-  (gr_line (start 156.86 114.46) (end 119.05 114.46) (layer Edge.Cuts) (width 0.1))
-  (gr_line (start 119.05 96.82) (end 119.05 114.46) (layer Edge.Cuts) (width 0.1))
-  (gr_line (start 150.1 96.82) (end 119.05 96.82) (layer Edge.Cuts) (width 0.1))
+  (gr_line (start 158.83 112.42) (end 156.83 114.42) (layer Edge.Cuts) (width 0.1))
+  (gr_line (start 158.83 98) (end 158.83 112.42) (layer Edge.Cuts) (width 0.1))
+  (gr_line (start 151.18 98) (end 158.83 98) (layer Edge.Cuts) (width 0.1))
+  (gr_line (start 151.18 107.3) (end 151.18 98) (layer Edge.Cuts) (width 0.1))
+  (gr_line (start 150.05 107.3) (end 151.18 107.3) (layer Edge.Cuts) (width 0.1))
+  (gr_line (start 150.05 96.87) (end 150.05 107.3) (layer Edge.Cuts) (width 0.1))
+  (gr_line (start 156.83 114.42) (end 119.1 114.42) (layer Edge.Cuts) (width 0.1))
+  (gr_line (start 119.1 96.87) (end 119.1 114.42) (layer Edge.Cuts) (width 0.1))
+  (gr_line (start 150.05 96.87) (end 119.1 96.87) (layer Edge.Cuts) (width 0.1))
   (gr_line (start 147.03 105) (end 147.03 112.89) (layer F.Fab) (width 0.127))
   (gr_line (start 141.48 109.35) (end 151.86 109.35) (layer F.Fab) (width 0.127))
@@
   (segment (start 151.7 110.18) (end 151.7 109.87) (width 0.2) (layer Back) (net 12))
   (zone (net 11) (net_name GND) (layer Front) (hatch edge 0.508)
-    (connect_pads (clearance 0.19))
-    (min_thickness 0.2)
-    (fill yes (arc_segments 32) (thermal_gap 0.4) (thermal_bridge_width 0.4))
+    (connect_pads (clearance 0.16))
+    (min_thickness 0.16)
+    (fill yes (arc_segments 32) (thermal_gap 0.25) (thermal_bridge_width 0.4))
     (polygon
       (pts
@@
   )
   (zone (net 11) (net_name GND) (layer Back) (hatch edge 0.508)
-    (connect_pads (clearance 0.19))
-    (min_thickness 0.2)
-    (fill yes (arc_segments 32) (thermal_gap 0.4) (thermal_bridge_width 0.4))
+    (connect_pads (clearance 0.16))
+    (min_thickness 0.16)
+    (fill yes (arc_segments 32) (thermal_gap 0.25) (thermal_bridge_width 0.5))
     (polygon
       (pts
